File: power.kicad_sch (KiCad schematic)
At the start: 0 parts

Commit message: [#51632] Power: add PoC circuit and description
Parts:
- added L?: L_15u_2.8A_Coilcraft-XAL4040, antmicro-footprints:L_Coilcraft-XAL4040, symbol antmicroFixedInductors:L_15u_2.8A_Coilcraft-XAL4040
- added R? (x2): R_5k1_0402, antmicro-footprints:R_0402_1005Metric, symbol antmicroResistors0402:R_5k1_0402
Connections:
- new net: L?.2, R?.1, R?.2
- new net +12V: L?.1, R?.1
Other:
- note added: "1812PS-22"
- note added: "MSS6132T-6"
- note added: "PFL1609-47N"
- note added: "PoC circuit C-6L-2000 as in GMSL2-hardware-design-guide GMSL 2 version Current Rating at Maximum Insertion Loss for 6G/187M : 2000mA @ 85C"
Changed lines of the file:
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@@
     (comment 1 "www.antmicro.com")
   )
+  (junction (at 62.23 50.8) (diameter 0) (color 0 0 0 0)
+  )
+  (junction (at 44.45 50.8) (diameter 0) (color 0 0 0 0)
+  )
+  (junction (at 62.23 60.325) (diameter 0) (color 0 0 0 0)
+  )
+  (junction (at 80.01 50.8) (diameter 0) (color 0 0 0 0)
+  )
+  (wire (pts (xy 38.1 50.8) (xy 44.45 50.8))
+    (stroke (width 0) (type default) (color 0 0 0 0))
+  )
+  (wire (pts (xy 50.8 60.325) (xy 44.45 60.325))
+    (stroke (width 0) (type default) (color 0 0 0 0))
+  )
+  (wire (pts (xy 80.01 60.325) (xy 80.01 50.8))
+    (stroke (width 0) (type default) (color 0 0 0 0))
+  )
+  (wire (pts (xy 44.45 50.8) (xy 50.8 50.8))
+    (stroke (width 0) (type default) (color 0 0 0 0))
+  )
+  (wire (pts (xy 73.66 60.325) (xy 80.01 60.325))
+    (stroke (width 0) (type default) (color 0 0 0 0))
+  )
+  (wire (pts (xy 127 50.8) (xy 139.7 50.8))
+    (stroke (width 0) (type default) (color 0 0 0 0))
+  )
+  (wire (pts (xy 55.88 60.325) (xy 62.23 60.325))
+    (stroke (width 0) (type default) (color 0 0 0 0))
+  )
+  (wire (pts (xy 62.23 50.8) (xy 68.58 50.8))
+    (stroke (width 0) (type default) (color 0 0 0 0))
+  )
+  (wire (pts (xy 44.45 60.325) (xy 44.45 50.8))
+    (stroke (width 0) (type default) (color 0 0 0 0))
+  )
+  (wire (pts (xy 62.23 60.325) (xy 62.23 50.8))
+    (stroke (width 0) (type default) (color 0 0 0 0))
+  )
+  (wire (pts (xy 68.58 60.325) (xy 62.23 60.325))
+    (stroke (width 0) (type default) (color 0 0 0 0))
+  )
+  (wire (pts (xy 144.78 50.8) (xy 151.13 50.8))
+    (stroke (width 0) (type default) (color 0 0 0 0))
+  )
+  (wire (pts (xy 91.44 50.8) (xy 104.14 50.8))
+    (stroke (width 0) (type default) (color 0 0 0 0))
+  )
+  (wire (pts (xy 109.22 50.8) (xy 121.92 50.8))
+    (stroke (width 0) (type default) (color 0 0 0 0))
+  )
+  (wire (pts (xy 80.01 50.8) (xy 86.36 50.8))
+    (stroke (width 0) (type default) (color 0 0 0 0))
+  )
+  (wire (pts (xy 80.01 50.8) (xy 73.66 50.8))
+    (stroke (width 0) (type default) (color 0 0 0 0))
+  )
+  (wire (pts (xy 62.23 50.8) (xy 55.88 50.8))
+    (stroke (width 0) (type default) (color 0 0 0 0))
+  )
+  (text "1812PS-22" (at 83.185 48.895 0)
+    (effects (font (size 1.27 1.27)) (justify left bottom))
+  )
+  (text "PFL1609-47N" (at 118.745 48.895 0)
+    (effects (font (size 1.27 1.27)) (justify left bottom))
+  )
+  (text "PFL1609-47N" (at 100.33 48.895 0)
+    (effects (font (size 1.27 1.27)) (justify left bottom))
+  )
+  (text "PoC circuit C-6L-2000 as in GMSL2-hardware-design-guide\nGMSL 2 version\nCurrent Rating at Maximum Insertion Loss for 6G/187M : 2000mA @ 85C\n"
+    (at 48.26 36.83 0)
+    (effects (font (size 1.27 1.27)) (justify left bottom))
+  )
+  (text "MSS6132T-6" (at 65.405 48.895 0)
+    (effects (font (size 1.27 1.27)) (justify left bottom))
+  )
+  (text "PFL1609-47N" (at 135.89 48.895 0)
+    (effects (font (size 1.27 1.27)) (justify left bottom))
+  )
+  (global_label "PoC" (shape output) (at 151.13 50.8 0) (fields_autoplaced)
+    (effects (font (size 1.27 1.27)) (justify left))
+    (property "Intersheet References" "${INTERSHEET_REFS}" (id 0) (at 157.2321 50.7206 0)
+      (effects (font (size 1.27 1.27)) (justify left) hide)
+    )
+  )
+  (symbol (lib_id "antmicroResistors0402:R_5k1_0402") (at 50.8 60.325 0) (unit 1)
+    (in_bom yes) (on_board yes) (fields_autoplaced)
+    (property "Reference" "R?" (id 0) (at 53.34 54.61 0)
+      (effects (font (size 1.27 1.27) (thickness 0.15)))
+    )
+    (property "Value" "R_5k1_0402" (id 1) (at 71.12 73.025 0)
+      (effects (font (size 1.27 1.27) (thickness 0.15)) (justify left bottom) hide)
+    )
+    (property "Footprint" "antmicro-footprints:R_0402_1005Metric" (id 2) (at 71.12 75.565 0)
+      (effects (font (size 1.27 1.27) (thickness 0.15)) (justify left bottom) hide)
+    )
+    (property "Datasheet" "https://www.bourns.com/docs/product-datasheets/cr.pdf" (id 3) (at 71.12 78.105 0)
+      (effects (font (size 1.27 1.27) (thickness 0.15)) (justify left bottom) hide)
+    )
+    (property "MPN" "CR0402-FX-5101GLF" (id 4) (at 71.12 80.645 0)
+      (effects (font (size 1.27 1.27) (thickness 0.15)) (justify left bottom) hide)
+    )
+    (property "Manufacturer" "Bourns" (id 5) (at 71.12 83.185 0)
+      (effects (font (size 1.27 1.27) (thickness 0.15)) (justify left bottom) hide)
+    )
+    (property "License" "Apache-2.0" (id 6) (at 71.12 85.725 0)
+      (effects (font (size 1.27 1.27) (thickness 0.15)) (justify left bottom) hide)
+    )
+    (property "Author" "Antmicro" (id 7) (at 71.12 88.265 0)
+      (effects (font (size 1.27 1.27) (thickness 0.15)) (justify left bottom) hide)
+    )
+    (property "Val" "5k1" (id 8) (at 53.34 57.15 0)
+      (effects (font (size 1.27 1.27) (thickness 0.15)))
+    )
+    (property "Tolerance" "1%" (id 9) (at 71.12 70.485 0)
+      (effects (font (size 1.27 1.27)) (justify left bottom) hide)
+    )
+    (pin "1")
+    (pin "2")
+  )
+  (symbol (lib_id "antmicropower:+12V") (at 38.1 50.8 0) (unit 1)
+    (in_bom yes) (on_board yes) (fields_autoplaced)
+    (property "Reference" "#PWR?" (id 0) (at 38.1 54.61 0)
+      (effects (font (size 1.27 1.27)) hide)
+    )
+    (property "Value" "+12V" (id 1) (at 38.1 45.72 0))
+    (property "Footprint" "" (id 2) (at 38.1 50.8 0)
+      (effects (font (size 1.27 1.27)) hide)
+    )
+    (property "Datasheet" "" (id 3) (at 38.1 50.8 0)
+      (effects (font (size 1.27 1.27)) hide)
+    )
+    (pin "1")
+  )
+  (symbol (lib_id "antmicroFixedInductors:L_15u_2.8A_Coilcraft-XAL4040") (at 50.8 50.8 0) (unit 1)
+    (in_bom yes) (on_board yes) (fields_autoplaced)
+    (property "Reference" "L?" (id 0) (at 53.34 45.72 0)
+      (effects (font (size 1.27 1.27) (thickness 0.15)))
+    )
+    (property "Value" "L_15u_2.8A_Coilcraft-XAL4040" (id 1) (at 66.04 60.96 0)
+      (effects (font (size 1.27 1.27) (thickness 0.15)) (justify left bottom) hide)
+    )
+    (property "Footprint" "antmicro-footprints:L_Coilcraft-XAL4040" (id 2) (at 66.04 63.5 0)
+      (effects (font (size 1.27 1.27) (thickness 0.15)) (justify left bottom) hide)
+    )
+    (property "Datasheet" "https://www.coilcraft.com/getmedia/6adcb47d-8b55-416c-976e-1e22e0d2848c/xal4000.pdf" (id 3) (at 66.04 66.04 0)
+      (effects (font (size 1.27 1.27) (thickness 0.15)) (justify left bottom) hide)
+    )
+    (property "Manufacturer" "Coilcraft" (id 4) (at 66.04 68.58 0)
+      (effects (font (size 1.27 1.27) (thickness 0.15)) (justify left bottom) hide)
+    )
+    (property "MPN" "XAL4040-153" (id 5) (at 66.04 71.12 0)
+      (effects (font (size 1.27 1.27) (thickness 0.15)) (justify left bottom) hide)
+    )
+    (property "ISat" "2.9 A" (id 6) (at 66.04 73.66 0)
+      (effects (font (size 1.27 1.27) (thickness 0.15)) (justify left bottom) hide)
+    )
+    (property "IMax" "2.8 A" (id 7) (at 66.04 76.2 0)
+      (effects (font (size 1.27 1.27) (thickness 0.15)) (justify left bottom) hide)
+    )
+    (property "Size" "4.0x4.0" (id 8) (at 66.04 78.74 0)
+      (effects (font (size 1.27 1.27) (thickness 0.15)) (justify left bottom) hide)
+    )
+    (property "Val" "15u/2.8A" (id 9) (at 53.34 48.26 0)
+      (effects (font (size 1.27 1.27) (thickness 0.15)))
+    )
+    (property "Author" "Antmicro" (id 10) (at 66.04 81.28 0)
+      (effects (font (size 1.27 1.27) (thickness 0.15)) (justify left bottom) hide)
+    )
+    (property "License" "Apache-2.0" (id 11) (at 66.04 83.82 0)
+      (effects (font (size 1.27 1.27) (thickness 0.15)) (justify left bottom) hide)
+    )
+    (pin "1")
+    (pin "2")
+  )
+  (symbol (lib_id "antmicroResistors0402:R_5k1_0402") (at 68.58 60.325 0) (unit 1)
+    (in_bom yes) (on_board yes) (fields_autoplaced)
+    (property "Reference" "R?" (id 0) (at 71.12 54.61 0)
+      (effects (font (size 1.27 1.27) (thickness 0.15)))
+    )
+    (property "Value" "R_5k1_0402" (id 1) (at 88.9 73.025 0)
+      (effects (font (size 1.27 1.27) (thickness 0.15)) (justify left bottom) hide)
+    )
+    (property "Footprint" "antmicro-footprints:R_0402_1005Metric" (id 2) (at 88.9 75.565 0)
+      (effects (font (size 1.27 1.27) (thickness 0.15)) (justify left bottom) hide)
+    )
+    (property "Datasheet" "https://www.bourns.com/docs/product-datasheets/cr.pdf" (id 3) (at 88.9 78.105 0)
+      (effects (font (size 1.27 1.27) (thickness 0.15)) (justify left bottom) hide)
+    )
+    (property "MPN" "CR0402-FX-5101GLF" (id 4) (at 88.9 80.645 0)
+      (effects (font (size 1.27 1.27) (thickness 0.15)) (justify left bottom) hide)
+    )
+    (property "Manufacturer" "Bourns" (id 5) (at 88.9 83.185 0)
+      (effects (font (size 1.27 1.27) (thickness 0.15)) (justify left bottom) hide)
+    )
+    (property "License" "Apache-2.0" (id 6) (at 88.9 85.725 0)
+      (effects (font (size 1.27 1.27) (thickness 0.15)) (justify left bottom) hide)
+    )
+    (property "Author" "Antmicro" (id 7) (at 88.9 88.265 0)
+      (effects (font (size 1.27 1.27) (thickness 0.15)) (justify left bottom) hide)
+    )
+    (property "Val" "5k1" (id 8) (at 71.12 57.15 0)
+      (effects (font (size 1.27 1.27) (thickness 0.15)))
+    )
+    (property "Tolerance" "1%" (id 9) (at 88.9 70.485 0)
+      (effects (font (size 1.27 1.27)) (justify left bottom) hide)
+    )
+    (pin "1")
+    (pin "2")
+  )
 )

Commit message: [#51632] Power: add current limit, buck conv Connectors: add buffer gates, remove one FFC conn
Parts:
- removed L?: L_15u_2.8A_Coilcraft-XAL4040, antmicro-footprints:L_Coilcraft-XAL4040, symbol antmicroFixedInductors:L_15u_2.8A_Coilcraft-XAL4040
- removed R? (x2): R_5k1_0402, antmicro-footprints:R_0402_1005Metric, symbol antmicroResistors0402:R_5k1_0402
- added C? (x4): C_10n_0402, antmicro-footprints:C_0402_1005Metric, symbol antmicroCapacitors0402:C_10n_0402
- added C? (x7): C_100n_0402, antmicro-footprints:C_0402_1005Metric, symbol antmicroCapacitors0402:C_100n_0402
- added C? (x4): C_22u_0402, antmicro-footprints:C_0402_1005Metric, symbol antmicroCapacitors0402:C_22u_0402
- added C? (x2): C_10u_25V_0603, antmicro-footprints:C_0603_1608Metric, symbol antmicroCapacitors0603:C_10u_25V_0603
- added L? (x2): L_1u_2.6A_0806, antmicro-footprints:L_0806_2016Metric, symbol antmicroFixedInductors:L_1u_2.6A_0806
- added Q?: BSS138AKA, antmicro-footprints:SOT-23-3, symbol antmicroTransistorsFETsMOSFETsSingle:BSS138AKA
- added Q?: BCM857BS-7-F, antmicro-footprints:SOT-363, symbol antmicroTransistorsBipolarArrays:BCM857BS-7-F
- added Q?: SQS401EN-T1_BE3, antmicro-footprints:Vishay_PowerPAK_1212-8_Single, symbol antmicroTransistorsFETsMOSFETsSingle:SQS401EN-T1_BE3
- added R? (x8): R_10k_0402, antmicro-footprints:R_0402_1005Metric, symbol antmicroResistors0402:R_10k_0402
- added R? (x2): R_100k_0402, antmicro-footprints:R_0402_1005Metric, symbol antmicroResistors0402:R_100k_0402
- added R? (x3): R_0R_22.4A_0603, antmicro-footprints:R_0603_1608Metric, symbol antmicroResistors0603:R_0R_22.4A_0603
- added R?: R_12k4_0402, antmicro-footprints:R_0402_1005Metric, symbol antmicroResistors0402:R_12k4_0402
- added R?: R_6k8_0402, antmicro-footprints:R_0402_1005Metric, symbol antmicroResistors0402:R_6k8_0402
- added R?: R_4k99_0402, antmicro-footprints:R_0402_1005Metric, symbol antmicroResistors0402:R_4k99_0402
- added R?: R_49R9_0402, antmicro-footprints:R_0402_1005Metric, symbol antmicroResistors0402:R_49R9_0402
- added U? (x2): AP62301_TSOT, antmicro-footprints:TSOT23-6, symbol antmicroDCDCConverters:AP62301_TSOT
- added U?: AP22615A_TSOT26, antmicro-footprints:TSOT23-6, symbol antmicroPMICPowerDistributionSwitchesLoadDrivers:AP22615A_TSOT26
- added U?: LMR62014XMF, antmicro-footprints:SOT-23-5, symbol antmicroDCDCConverters:LMR62014XMF
Connections:
- net +12V: now also C?.2, C?.2, C?.2, C?.2, C?.2, C?.2, C?.2, C?.2, C?.2, C?.2, Q?.1, Q?.1 (S), R?.2, R?.2, R?.2, U?.3 (VIN), U?.3 (VIN)
- new net: Q?.4 (G), Q?.6, R?.2
- new net: Q?.1 (G), R?.2, R?.2
- new net: C?.1, U?.6 (BST) (x2)
- new net: Q?.2, Q?.3, Q?.5, R?.2
- new net +1V2: R?.2
- new net +1V8: R?.2, R?.2, R?.2
- new net +5V: U?.1 (OUT)
- new net DC_IN: Q?.4, Q?.5 (D), R?.1, R?.1
- new net EN_1V2: R?.1, U?.5 (EN)
- new net EN_1V8: R?.1, U?.5 (EN)
- new net FB_1V2: R?.1, R?.2, U?.4 (FB)
- new net FB_1V8: R?.1, R?.2, U?.4 (FB)
- new net FFC_5V: C?.2, U?.6 (IN)
- new net FFC_5V_EN: Q?.3 (D), R?.1, R?.2, U?.4 (EN)
- new net FFC_5V_FLG: R?.1, U?.3 (FLG)
- new net FFC_5V_ISET: R?.2, U?.5 (ISET)
- new net GND: C?.1, C?.1, C?.1, C?.1, C?.1, C?.1, C?.1, C?.1, C?.1, C?.1, C?.1, C?.1, C?.1, C?.1, C?.1, Q?.2 (S), R?.1, R?.1, R?.1, R?.1, R?.1, R?.1, R?.1, U?.1 (GND), U?.1 (GND), U?.2 (GND)
- new net OUT_1V2: C?.2, C?.2, L?.2, R?.1, R?.2
- new net OUT_1V8: C?.2, C?.2, L?.2, R?.1, R?.2
- new net SW_1V2: C?.2, L?.1, U?.2 (SW)
- new net SW_1V8: C?.2, L?.1, U?.2 (SW)
Other:
- note added: "FFC 5V current limit"
- note added: "PoC circuit"
- note added: "Power supply"
- note added: "TODO: booster 5=>12V power arbiter"
- note removed: "1812PS-22"
- note removed: "MSS6132T-6"
- note removed: "PFL1609-47N"
- note removed: "PoC circuit C-6L-2000 as in GMSL2-hardware-design-guide GMSL 2 version Current Rating at Maximum Insertion Loss for 6G/187M : 2000mA @ 85C"

Commit message: Schematics done
Parts:
- added C14: C_2u2_0402, antmicro-footprints:C_0402_1005Metric, symbol antmicroCapacitors0402:C_2u2_0402
- added C15: C_220p_0402, antmicro-footprints:C_0402_1005Metric, symbol antmicroCapacitors0402:C_220p_0402
- added C16: C_10u_25V_0603, antmicro-footprints:C_0603_1608Metric, symbol antmicroCapacitors0603:C_10u_25V_0603
- added D3: PMEG3010CE_SOD323, antmicro-footprints:D_SOD-323F, symbol antmicroDiodesRectifiersSingle:PMEG3010CE_SOD323
- added L1, L2, L3, L4: L_22u_1.12A_Coilcraft-MSS6132T, antmicro-footprints:L_Coilcraft-MSS6132T, symbol antmicroFixedInductors:L_22u_1.12A_Coilcraft-MSS6132T
- added L10, L11, L12, L13, L14, L15, L16, L9: L_470n_1A_Coilcraft-PFL1609, antmicro-footprints:L_Coilcraft-PFL1609, symbol antmicroFixedInductors:L_470n_1A_Coilcraft-PFL1609
- added L17: L_10u_3.1A_Bourns-SRN8040, antmicro-footprints:L_Bourns-SRN8040, symbol antmicroFixedInductors:L_10u_3.1A_Bourns-SRN8040
- added L5, L6, L7, L8: L_6u8_1A_Coilcraft-1210POC, antmicro-footprints:L_Coilcraft-1210POC, symbol antmicroFixedInductors:L_6u8_1A_Coilcraft-1210POC
- added R19, R20, R21, R22, R24, R25, R26, R27: R_5k1_0402, antmicro-footprints:R_0402_1005Metric, symbol antmicroResistors0402:R_5k1_0402
- added R28: R_51k_0402, antmicro-footprints:R_0402_1005Metric, symbol antmicroResistors0402:R_51k_0402
- added R29: R_13k7_0402, antmicro-footprints:R_0402_1005Metric, symbol antmicroResistors0402:R_13k7_0402
- added R30: R_120k_0402, antmicro-footprints:R_0402_1005Metric, symbol antmicroResistors0402:R_120k_0402
- gave numbers to parts that had none: 43
Connections:
- net +12V: now also C15.2, C16.2, D3.K, L1.1, L2.1, L3.1, L4.1, R19.1, R20.1, R21.1, R22.1, R30.2
- net +5V: now also U3.5 (VIN), C14.2, L17.1, R28.2
- net GND: now also U3.2 (GND), C14.1, C16.1, R29.1
- net PoCA: now also L13.2
- net PoCB: now also L14.2
- net PoCC: now also L15.2
- net PoCD: now also L16.2
- net at U3.1 (SW): now also D3.A, L17.2
- net at U3.3 (FB): now also C15.1, R29.2, R30.1
- net at U3.4 (~{SHDN}): now also R28.1
- new net: L4.2, L8.1, R22.2, R27.1
- new net: L12.1, L8.2, R27.2
- new net: L2.2, L6.1, R20.2, R25.1
- new net: L3.2, L7.1, R21.2, R26.1
- new net: L1.2, L5.1, R19.2, R24.1
- new net: L10.1, L6.2, R25.2
- new net: L5.2, L9.1, R24.2
- new net: L11.2, L15.1
- new net: L11.1, L7.2, R26.2
- new net: L10.2, L14.1
- new net: L13.1, L9.2
- new net: L12.2, L16.1
Other:
- note added: "Boost converter 5V to 12V"
- note added: "Buck converter 12V to 1.2V"
- note added: "Buck converter 12V to 1.8V"
- note added: "Power arbiter"
- note removed: "Power supply"
- note removed: "TODO: booster 5=>12V power arbiter"
- moved on the sheet: C18, C20, C22, C25, L19, R31, R37, R38, R41, U3, U5
