File: gmsl-deserializer.kicad_sch (KiCad schematic)
At the start: 6 parts

Commit message: [#55438] Update symbols and footprints, clean ERC and DRC
Parts:
- removed N1: oshw_logo, antmicro-footprints:oshw-logo, symbol antmicroMechanicalParts:oshw_logo
- removed N2: antmicro_logo, antmicro-footprints:antmicro-logo_scaled_12mm, symbol antmicroMechanicalParts:antmicro_logo
Other:
- moved on the sheet: H1, H3
