File: deserializer.kicad_sch (KiCad schematic)
At the start: 49 parts, among them U7 MAX96724GTN_VY+, Y1 Resonator_25MHz_ABM8G

Commit message: [#74135] Fix DNP malformations
Parts:
- R48, R50: DNP DNP -> (none)
Changed lines of the file:
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@@
-			)
-		)
-		(property "DNP" "DNP"
-			(at 121.92 180.34 0)
-			(effects
-				(font
-					(size 1.27 1.27)
-				)
-				(hide yes)
 			)
 		)
@@
 				(hide yes)
 			)
-		)
-		(property "DNP" "DNP"
-			(at 162.56 180.34 0)
-			(effects
-				(font
-					(size 1.27 1.27)
-				)
-				(hide yes)
-			)
